Commit message: Added handle to fridge door

File: popcanbot_description/urdf/fridge.xacro (robot description, xacro)
@@ -5,4 +5,8 @@
 <xacro:property name="height" value="0.7"/>
 <xacro:property name="wall_thickness" value="0.05"/>
+<xacro:property name="handle_length" value="0.06"/>
+<xacro:property name="handle_width" value="0.03"/>
+<xacro:property name="handle_height" value="0.1"/>
+<xacro:property name="handle_thickness" value="0.025"/>
 <xacro:include filename="$(find popcanbot_description)/urdf/util.xacro"/>
   <link name="fridge_base_link"/>
@@ -66,3 +70,11 @@
     <limit effort="100.0" upper="2.5" lower="0" velocity="0.5"/>
   </joint>
+  <xacro:block name="handle_front" length="${handle_thickness}"
+      width="${handle_width}" height="${handle_height}" mass="0.1"
+      r="1.0" g="1.0" b="1.0"/>
+  <joint name="handle_front_joint" type="fixed">
+    <parent link="fridge_door"/>
+    <child link="handle_front"/>
+    <origin xyz="${handle_length + wall_thickness/2} ${-width + handle_width/2} 0" rpy="0 0 0"/>
+  </joint>
 </robot>

Commit message: Making can spawn inside fridge #2 is only reliably done with pause set to true, also adjusting spawn parameters, and making fridge door not open without a bit of effort, and making this work in jade.

File: popcanbot_description/urdf/fridge.xacro (robot description, xacro)
@@ -66,7 +66,9 @@
     <parent link="fridge_bottom"/>
     <child link="fridge_door"/>
-    <origin xyz="${length/2} ${width/2} ${height/2}" rpy="0 0 0"/>
+    <!-- tilt the door very slightly so it doesn't fall open  -->
+    <origin xyz="${length/2} ${width/2} ${height/2}" rpy="0 -0.001 0"/>
+    <dynamics damping="0.1" friction="0.1"/>
     <axis xyz="0 0 1"/>
-    <limit effort="100.0" upper="2.5" lower="0" velocity="0.5"/>
+    <limit effort="10.0" upper="2.5" lower="0" velocity="0.1"/>
   </joint>
   <xacro:block name="handle_front" length="${handle_thickness}"

File: popcanbot_description/urdf/util.xacro (robot description, xacro)
@@ -63,5 +63,6 @@
   </link>
   <gazebo reference="${name}">
-    <color rgba="${r} ${g} ${b} 1.0"/>
+    <!-- this doesn't work, how to specify rgb color for gazebo? -->
+    <!--color rgba="${r} ${g} ${b} 1.0"/-->
   </gazebo>
 </xacro:macro>

Commit message: Tuning parameters and adding ui rqt window

File: popcanbot_description/urdf/fridge.xacro (robot description, xacro)
@@ -11,6 +11,6 @@
 <xacro:include filename="$(find popcanbot_description)/urdf/util.xacro"/>
   <link name="fridge_base_link"/>
-  <xacro:block name="fridge_bottom" length="${length}"
-      width="${width}" height="${wall_thickness}" mass="5.0"
+  <xacro:block name="fridge_bottom" length="${length * 0.98}"
+      width="${width * 0.98}" height="${wall_thickness}" mass="5.0"
       r="0.7" g="0.7" b="0.7"/>
   <joint name="bottom_joint" type="fixed">
@@ -43,6 +43,6 @@
     <origin xyz="0 ${-width/2} ${height/2}" rpy="0 0 0"/>
   </joint>
-  <xacro:block name="fridge_shelf" length="${length}"
-      width="${width}" height="${wall_thickness}" mass="5.0"
+  <xacro:block name="fridge_shelf" length="${length * 0.98}"
+      width="${width * 0.98}" height="${wall_thickness * 0.9}" mass="5.0"
       r="0.7" g="0.7" b="0.7"/>
   <joint name="shelf_joint" type="fixed">
@@ -51,6 +51,6 @@
     <origin xyz="0 0 ${height/2}" rpy="0 0 0"/>
   </joint>
-  <xacro:block name="fridge_top" length="${length}"
-      width="${width}" height="${wall_thickness}" mass="5.0"
+  <xacro:block name="fridge_top" length="${length * 0.98}"
+      width="${width * 0.98}" height="${wall_thickness}" mass="5.0"
       r="0.7" g="0.7" b="0.7"/>
   <joint name="top_joint" type="fixed">

File: popcanbot_description/urdf/popcanbot.xacro (robot description, xacro)
@@ -66,4 +66,5 @@
     <axis xyz="0 0 1"/>
     <limit effort="100.0" upper="1.6" lower="-1.6" velocity="0.5"/>
+    <dynamics damping="0.1" friction="0.1"/>
   </joint>
   <transmission name="arm_vertical_rotary_tran">
@@ -85,5 +86,6 @@
     <origin xyz="0.05 0 0.25" rpy="0 0 0"/>
     <axis xyz="0 0 1"/>
-    <limit effort="20.0" velocity="0.25" lower="-0.14" upper="0.30"/>
+    <limit effort="20.0" velocity="0.25" lower="-0.14" upper="0.35"/>
+    <dynamics damping="0.1" friction="0.1"/>
   </joint>
   <transmission name="arm_vertical_rotary_tran">
@@ -105,4 +107,5 @@
     <axis xyz="1 0 0"/>
     <limit effort="20.0" velocity="0.25" lower="-0.22" upper="0.05"/>
+    <dynamics damping="0.1" friction="0.1"/>
   </joint>
   <transmission name="arm_vertical_rotary_tran">
@@ -124,5 +127,6 @@
     <origin xyz="0.25 0.02 -0.1" rpy="0 0 0"/>
     <axis xyz="0 0 1"/>
-    <limit effort="100.0" upper="0.7" lower="-0.1" velocity="0.5"/>
+    <limit effort="200.0" upper="0.7" lower="-0.1" velocity="0.5"/>
+    <dynamics damping="0.1" friction="0.1"/>
   </joint>
   <xacro:block name="gripper_left_mid" length="0.07"
@@ -157,7 +161,8 @@
     <origin xyz="0.25 -0.02 -0.1" rpy="0 0 0"/>
     <axis xyz="0 0 1"/>
-    <limit effort="100.0" upper="0.1" lower="-0.4" velocity="0.5"/>
+    <limit effort="200.0" upper="0.1" lower="-0.5" velocity="0.5"/>
+    <dynamics damping="0.1" friction="0.1"/>
     <!-- mimic doesn't do anything in gazebo, but should be useful in pure rviz -->
-    <mimic joint="gripper_left_joint" multiplier="-1.0"/>
+    <!--mimic joint="gripper_left_joint" multiplier="-1.0"/-->
   </joint>
   <xacro:block name="gripper_right_mid" length="0.07"
@@ -190,9 +195,10 @@
       width="0.02" height="0.03" mass="0.1"/>
   <joint name="camera_mast_joint" type="prismatic">
-    <parent link="base_link"/>
+    <parent link="arm_horizontal"/>
     <child link="camera_mast"/>
-    <origin xyz="0.1 0 0.4" rpy="0 0 0"/>
+    <origin xyz="0.1 0 0.2" rpy="0 0 0"/>
     <axis xyz="0 0 1"/>
     <limit effort="20.0" velocity="0.25" lower="0.0" upper="0.5"/>
+    <dynamics damping="0.1" friction="0.1"/>
   </joint>
   <xacro:block name="camera_link" length="0.05"
