Commit message: Capturing essential mechanism in arm, but need to modify grippers to actually grip, and wheels aren't right to make the robot level

File: popcanbot_description/urdf/popcanbot.xacro (robot description, xacro)
@@ -1,9 +1,10 @@
 <?xml version="1.0"?>
 <robot name="popcanbot" xmlns:xacro="http://wiki.ros.org/xacro">
-<xacro:property name="car_length" value="1.4"/>
-<xacro:property name="car_width" value="1.0"/>
-<xacro:property name="car_height" value="0.3"/>
-<xacro:property name="wheel_width" value="0.15"/>
-<xacro:property name="wheel_radius" value="0.2"/>
+<xacro:property name="car_length" value="0.609"/>
+<xacro:property name="car_width" value="0.5"/>
+<xacro:property name="car_height" value="0.05"/>
+<xacro:property name="wheel_width" value="0.025"/>
+<xacro:property name="wheel_radius" value="0.07"/>
+<xacro:property name="use_camera" value="false"/>
 <!-- TODO(lwalter) pass these in as args -->
 <xacro:include filename="$(find popcanbot_description)/urdf/popcanbot.gazebo"/>
@@ -11,8 +12,9 @@
   like 'box', 'cylinder', etc. otherwise get Invalid parameter "size"
 -->
-<xacro:macro name="block" params="name length width height mass r:=0.5 b:=0.5 g:=0.5">
+<xacro:macro name="block" params="name length width height mass
+    x:=0 y:=0 z:=0 r:=0.5 b:=0.5 g:=0.5">
   <link name="${name}">
      <visual>
-      <origin xyz="0 0 0" rpy="0 0 0"/>
+      <origin xyz="${x} ${y} ${z}" rpy="0 0 0"/>
       <geometry>
         <box size="${length} ${width} ${height}"/>
@@ -23,5 +25,5 @@
     </visual>
     <collision>
-      <origin xyz="0 0 0" rpy="0 0 0" />
+      <origin xyz="${x} ${y} ${z}" rpy="0 0 0"/>
       <geometry>
         <box size="${length} ${width} ${height}"/>
@@ -29,5 +31,5 @@
     </collision>
     <inertial>
-      <origin xyz="0 0 0" rpy="0 0 0" />
+      <origin xyz="${x} ${y} ${z}" rpy="0 0 0"/>
       <mass value="${mass}"/>
       <inertia
@@ -95,5 +97,5 @@
 <!-- TODO(lucasw) make a wheel xacro to get common code out of
     fixed_wheel and steered_wheel -->
-<xacro:macro name="fixed_wheel" params="name parent y">
+<xacro:macro name="fixed_wheel" params="name parent y radius">
   <xacro:block name="${name}" length="${car_width/8.0}"
       width="${car_width/8.0}" height="${car_width/8.0}" mass="0.1"/>
@@ -104,9 +106,10 @@
   </joint>
   <xacro:generic_wheel name="${name}" parent="${name}"
-      radius="${wheel_radius}" width="${wheel_width}"/>
+      radius="${radius}" width="${wheel_width}"/>
  </xacro:macro>
   <link name="base_link"/>
   <xacro:block name="chassis_link" length="${car_length}"
-      width="${car_width}" height="${car_height}" mass="10.0"/>
+      width="${car_width}" height="${car_height}" mass="10.0"
+      r="0.8" g="0.7" b="0.1"/>
   <joint name="chassis_joint" type="fixed">
     <parent link="base_link"/>
@@ -127,5 +130,5 @@
   </joint>
   <xacro:fixed_wheel name="caster" parent="caster_block"
-      y="0"/>
+      y="0" radius="${wheel_radius * 0.5}"/>
   <xacro:block name="main_axle" length="${car_width/8.0}"
       width="${car_width}" height="${car_width/8.0}" mass="0.1"/>
@@ -133,11 +136,70 @@
     <parent link="base_link"/>
     <child link="main_axle"/>
-    <origin xyz="${car_length/2 - 0.1} 0 0" rpy="0 0 0"/>
+    <origin xyz="${car_length/2 - 0.1} 0 ${-car_height/4}" rpy="0 0 0"/>
   </joint>
   <xacro:fixed_wheel name="back_left" parent="main_axle"
-      y="${car_width/2 + wheel_width/2 + 0.1}"/>
+      y="${car_width/2 + wheel_width/2 + 0.1}" radius="${wheel_radius}"/>
   <xacro:fixed_wheel name="back_right" parent="main_axle"
-      y="${-1 * (car_width/2 + wheel_width/2 + 0.1)}"/>
+      y="${-1 * (car_width/2 + wheel_width/2 + 0.1)}" radius="${wheel_radius}"/>
+  <!-- the arm -->
+  <xacro:block name="arm_vertical" length="0.05"
+      width="0.05" height="0.5" mass="1.0" z="0.25"/>
+  <joint name="arm_vertical_rotary_joint" type="revolute">
+    <parent link="base_link"/>
+    <child link="arm_vertical"/>
+    <origin xyz="0 0 ${car_height/4}" rpy="0 0 0"/>
+    <axis xyz="0 0 1"/>
+    <limit effort="100.0" upper="1.6" lower="-1.6" velocity="0.5"/>
+  </joint>
+  <transmission name="arm_vertical_rotary_tran">
+    <type>transmission_interface/SimpleTransmission</type>
+    <joint name="arm_vertical_rotary_joint">
+      <hardwareInterface>EffortJointInterface</hardwareInterface>
+    </joint>
+    <actuator name="arm_vertical_rotary_motor">
+      <hardwareInterface>EffortJointInterface</hardwareInterface>
+      <mechanicalReduction>1</mechanicalReduction>
+    </actuator>
+  </transmission>
+  <xacro:block name="arm_vertical_platform" length="0.05"
+      width="0.1" height="0.05" mass="0.1"
+      r="0.8" g="0.8" b="0.8"/>
+  <joint name="arm_vertical_platform" type="prismatic">
+    <parent link="arm_vertical"/>
+    <child link="arm_vertical_platform"/>
+    <origin xyz="0.05 0 0.25" rpy="0 0 0"/>
+    <axis xyz="0 0 1"/>
+    <limit effort="20.0" velocity="0.25" lower="-0.20" upper="0.20"/>
+  </joint>
+  <xacro:block name="arm_horizontal" length="0.5"
+      width="0.05" height="0.05" mass="0.2"/>
+  <joint name="arm_horizontal_platform" type="prismatic">
+    <parent link="arm_vertical_platform"/>
+    <child link="arm_horizontal"/>
+    <origin xyz="0.1 -0.06 -0.05" rpy="0 0 0"/>
+    <axis xyz="1 0 0"/>
+    <limit effort="20.0" velocity="0.25" lower="-0.22" upper="0.05"/>
+  </joint>
+  <!-- gripper -->
+  <xacro:block name="gripper_left" length="0.07"
+      width="0.02" height="0.02" mass="0.05" r="0.1" b="0.1" g="0.6" x="0.03"/>
+  <joint name="gripper_left_joint" type="revolute">
+    <parent link="arm_horizontal"/>
+    <child link="gripper_left"/>
+    <origin xyz="0.25 0.015 -0.05" rpy="0 0 0"/>
+    <axis xyz="0 0 1"/>
+    <limit effort="100.0" upper="0.4" lower="-0.1" velocity="0.5"/>
+  </joint>
+  <xacro:block name="gripper_right" length="0.07"
+      width="0.02" height="0.02" mass="0.05" r="0.1" b="0.1" g="0.6" x="0.03"/>
+  <joint name="gripper_right_joint" type="revolute">
+    <parent link="arm_horizontal"/>
+    <child link="gripper_right"/>
+    <origin xyz="0.25 -0.015 -0.05" rpy="0 0 0"/>
+    <axis xyz="0 0 1"/>
+    <limit effort="100.0" upper="0.1" lower="-0.4" velocity="0.5"/>
+  </joint>
   <!-- sensors -->
+  <xacro:if value="${use_camera}">
   <xacro:block name="camera_mast" length="0.04"
       width="0.02" height="0.03" mass="0.1"/>
@@ -166,3 +228,4 @@
     <child link="camera_link_optical"/>
   </joint>
+  </xacro:if>
 </robot>

Commit message: Grippers have bend in them that might be able to grip things in gazebo.

File: popcanbot_description/urdf/popcanbot.xacro (robot description, xacro)
@@ -4,6 +4,8 @@
 <xacro:property name="car_width" value="0.5"/>
 <xacro:property name="car_height" value="0.05"/>
+<xacro:property name="clearance" value="0.10"/>
 <xacro:property name="wheel_width" value="0.025"/>
 <xacro:property name="wheel_radius" value="0.07"/>
+<xacro:property name="caster_wheel_radius" value="0.04"/>
 <xacro:property name="use_camera" value="false"/>
 <!-- TODO(lwalter) pass these in as args -->
@@ -69,16 +71,18 @@
   </link>
 </xacro:macro>
-<xacro:macro name="generic_wheel" params="name parent radius width">
-  <xacro:wheel name="wheel_${name}" width="${wheel_width}" radius="${wheel_radius}" mass="0.2"/>
-  <joint name="wheel_${name}_axle" type="continuous">
+<xacro:macro name="generic_wheel" params="name parent radius width
+    z:=0 y:=0 y_axis:=1 mass:=0.2 use_tran:=true">
+  <xacro:wheel name="${name}" width="${width}" radius="${radius}" mass="${mass}"/>
+  <joint name="${name}_joint" type="continuous">
     <parent link="${parent}"/>
-    <child link="wheel_${name}"/>
-    <origin xyz="0 0 ${-car_height/4}" rpy="0 0 0"/>
-    <axis xyz="0 1 0"/>
+    <child link="${name}"/>
+    <origin xyz="0 ${y} ${z}" rpy="0 0 0"/>
+    <axis xyz="0 ${y_axis} 0"/>
     <limit effort="100.0" velocity="0.5"/>
   </joint>
+  <xacro:if value="${use_tran}">
   <transmission name="${name}_tran">
     <type>transmission_interface/SimpleTransmission</type>
-    <joint name="wheel_${name}_axle">
+    <joint name="${name}_joint">
       <hardwareInterface>EffortJointInterface</hardwareInterface>
     </joint>
@@ -88,4 +92,5 @@
     </actuator>
   </transmission>
+  </xacro:if>
   <gazebo reference="wheel_${name}">
     <mu1>800</mu1>
@@ -95,17 +100,4 @@
   </gazebo>
 </xacro:macro>  <!-- generic wheel -->
-<!-- TODO(lucasw) make a wheel xacro to get common code out of
-    fixed_wheel and steered_wheel -->
-<xacro:macro name="fixed_wheel" params="name parent y radius">
-  <xacro:block name="${name}" length="${car_width/8.0}"
-      width="${car_width/8.0}" height="${car_width/8.0}" mass="0.1"/>
-  <joint name="${name}_axle" type="fixed">
-    <parent link="${parent}"/>
-    <child link="${name}"/>
-    <origin xyz="0 ${y} 0" rpy="0 0 0"/>
-  </joint>
-  <xacro:generic_wheel name="${name}" parent="${name}"
-      radius="${radius}" width="${wheel_width}"/>
- </xacro:macro>
   <link name="base_link"/>
   <xacro:block name="chassis_link" length="${car_length}"
@@ -121,25 +113,32 @@
     that doesn't have inertia won't appear.
     -->
-  <xacro:block name="caster_block" length="${car_width/8.0}"
-      width="${car_width/8.0}" height="${car_width/8.0}" mass="0.1"/>
+  <xacro:block name="caster_block" length="${0.03}"
+      width="${0.03}" height="${0.03}" mass="0.1"/>
   <joint name="caster_joint" type="continuous">
     <parent link="base_link"/>
     <child link="caster_block"/>
     <axis xyz="0 0 1"/>
-    <origin xyz="${-car_length/2 + 0.1} 0 -0.1" rpy="0 0 0"/>
-  </joint>
-  <xacro:fixed_wheel name="caster" parent="caster_block"
-      y="0" radius="${wheel_radius * 0.5}"/>
+    <origin xyz="${-car_length/2 + 0.1} 0 ${-car_height/2}" rpy="0 0 0"/>
+  </joint>
+  <xacro:generic_wheel name="wheel_caster" parent="caster_block"
+      width="${wheel_width}"
+      radius="${caster_wheel_radius}" mass="0.1" use_tran="false"
+      z="${-(clearance - caster_wheel_radius)}"/>
   <xacro:block name="main_axle" length="${car_width/8.0}"
-      width="${car_width}" height="${car_width/8.0}" mass="0.1"/>
+      width="${car_width + 0.05}" height="${car_width/8.0}" mass="0.1"
+      />
   <joint name="main_axle_joint" type="fixed">
     <parent link="base_link"/>
     <child link="main_axle"/>
-    <origin xyz="${car_length/2 - 0.1} 0 ${-car_height/4}" rpy="0 0 0"/>
-  </joint>
-  <xacro:fixed_wheel name="back_left" parent="main_axle"
-      y="${car_width/2 + wheel_width/2 + 0.1}" radius="${wheel_radius}"/>
-  <xacro:fixed_wheel name="back_right" parent="main_axle"
-      y="${-1 * (car_width/2 + wheel_width/2 + 0.1)}" radius="${wheel_radius}"/>
+    <origin xyz="${car_length/2 - 0.1} 0 ${-(car_height/2 + clearance - wheel_radius)}"
+        rpy="0 0 0"/>
+  </joint>
+  <xacro:generic_wheel name="wheel_front_left" parent="main_axle"
+      y="${car_width/2 + wheel_width/2 + 0.1}"
+      width="${wheel_width}" radius="${wheel_radius}"/>
+  <xacro:generic_wheel name="wheel_front_right" parent="main_axle"
+      y="${-1 * (car_width/2 + wheel_width/2 + 0.1)}"
+      width="${wheel_width}" radius="${wheel_radius}"
+      y_axis="1"/>
   <!-- the arm -->
   <xacro:block name="arm_vertical" length="0.05"
@@ -187,7 +186,14 @@
     <parent link="arm_horizontal"/>
     <child link="gripper_left"/>
-    <origin xyz="0.25 0.015 -0.05" rpy="0 0 0"/>
+    <origin xyz="0.25 0.02 -0.05" rpy="0 0 0"/>
     <axis xyz="0 0 1"/>
     <limit effort="100.0" upper="0.4" lower="-0.1" velocity="0.5"/>
+  </joint>
+  <xacro:block name="gripper_left_tip" length="0.07"
+      width="0.02" height="0.02" mass="0.05" r="0.1" b="0.1" g="0.6" x="0.03"/>
+  <joint name="gripper_left_tip_joint" type="fixed">
+    <parent link="gripper_left"/>
+    <child link="gripper_left_tip"/>
+    <origin xyz="0.05 0.0 0.0" rpy="0 0 -0.3"/>
   </joint>
   <xacro:block name="gripper_right" length="0.07"
@@ -196,7 +202,14 @@
     <parent link="arm_horizontal"/>
     <child link="gripper_right"/>
-    <origin xyz="0.25 -0.015 -0.05" rpy="0 0 0"/>
+    <origin xyz="0.25 -0.02 -0.05" rpy="0 0 0"/>
     <axis xyz="0 0 1"/>
     <limit effort="100.0" upper="0.1" lower="-0.4" velocity="0.5"/>
+  </joint>
+  <xacro:block name="gripper_right_tip" length="0.07"
+      width="0.02" height="0.02" mass="0.05" r="0.1" b="0.1" g="0.6" x="0.03"/>
+  <joint name="gripper_right_tip_joint" type="fixed">
+    <parent link="gripper_right"/>
+    <child link="gripper_right_tip"/>
+    <origin xyz="0.05 0.0 0.0" rpy="0 0 0.3"/>
   </joint>
   <!-- sensors -->

Commit message: The robot is getting loaded into gazebo now.

File: popcanbot_description/urdf/popcanbot.xacro (robot description, xacro)
@@ -135,8 +135,8 @@
   </joint>
   <xacro:generic_wheel name="wheel_front_left" parent="main_axle"
-      y="${car_width/2 + wheel_width/2 + 0.1}"
+      y="${car_width/2 + wheel_width/2 + 0.02}"
       width="${wheel_width}" radius="${wheel_radius}"/>
   <xacro:generic_wheel name="wheel_front_right" parent="main_axle"
-      y="${-1 * (car_width/2 + wheel_width/2 + 0.1)}"
+      y="${-1 * (car_width/2 + wheel_width/2 + 0.02)}"
       width="${wheel_width}" radius="${wheel_radius}"
       y_axis="1"/>
@@ -169,5 +169,5 @@
     <origin xyz="0.05 0 0.25" rpy="0 0 0"/>
     <axis xyz="0 0 1"/>
-    <limit effort="20.0" velocity="0.25" lower="-0.20" upper="0.20"/>
+    <limit effort="20.0" velocity="0.25" lower="-0.14" upper="0.20"/>
   </joint>
   <xacro:block name="arm_horizontal" length="0.5"

Commit message: Added controllers and tuned pid parameters for rest of joints except gripper (try out a mirror joint there?).  The wheels really need velocity controllers, or my own controller to send a continuous stream of smoother intermediate positions when given a desired velocity

File: popcanbot_description/urdf/popcanbot.xacro (robot description, xacro)
@@ -164,5 +164,5 @@
       width="0.1" height="0.05" mass="0.1"
       r="0.8" g="0.8" b="0.8"/>
-  <joint name="arm_vertical_platform" type="prismatic">
+  <joint name="arm_vertical_platform_joint" type="prismatic">
     <parent link="arm_vertical"/>
     <child link="arm_vertical_platform"/>
@@ -171,7 +171,17 @@
     <limit effort="20.0" velocity="0.25" lower="-0.14" upper="0.20"/>
   </joint>
+  <transmission name="arm_vertical_rotary_tran">
+    <type>transmission_interface/SimpleTransmission</type>
+    <joint name="arm_vertical_platform_joint">
+      <hardwareInterface>EffortJointInterface</hardwareInterface>
+    </joint>
+    <actuator name="arm_vertical_platform_motor">
+      <hardwareInterface>EffortJointInterface</hardwareInterface>
+      <mechanicalReduction>1</mechanicalReduction>
+    </actuator>
+  </transmission>
   <xacro:block name="arm_horizontal" length="0.5"
       width="0.05" height="0.05" mass="0.2"/>
-  <joint name="arm_horizontal_platform" type="prismatic">
+  <joint name="arm_horizontal_platform_joint" type="prismatic">
     <parent link="arm_vertical_platform"/>
     <child link="arm_horizontal"/>
@@ -180,4 +190,14 @@
     <limit effort="20.0" velocity="0.25" lower="-0.22" upper="0.05"/>
   </joint>
+  <transmission name="arm_vertical_rotary_tran">
+    <type>transmission_interface/SimpleTransmission</type>
+    <joint name="arm_horizontal_platform_joint">
+      <hardwareInterface>EffortJointInterface</hardwareInterface>
+    </joint>
+    <actuator name="arm_horizontal_platform_motor">
+      <hardwareInterface>EffortJointInterface</hardwareInterface>
+      <mechanicalReduction>1</mechanicalReduction>
+    </actuator>
+  </transmission>
   <!-- gripper -->
   <xacro:block name="gripper_left" length="0.07"

Commit message: Now have crude rendition of http://www.robothon.org/robothon/images/contest/popcanarena_diagram.pdf in gazebo, there are some neat pre-existing kitchen and house models with chairs and refrigerators but the models are all integrated- need to get in with a text editor to extract anything, the gazebo gui can't do it.

File: popcanbot_description/urdf/popcanbot.xacro (robot description, xacro)
@@ -8,5 +8,5 @@
 <xacro:property name="wheel_radius" value="0.07"/>
 <xacro:property name="caster_wheel_radius" value="0.04"/>
-<xacro:property name="use_camera" value="false"/>
+<xacro:property name="use_camera" value="true"/>
 <!-- TODO(lwalter) pass these in as args -->
 <xacro:include filename="$(find popcanbot_description)/urdf/popcanbot.gazebo"/>

Commit message: Now have a basic fridge model, get this into gazebo and get the pop can into it

File: popcanbot_description/urdf/popcanbot.xacro (robot description, xacro)
@@ -11,93 +11,5 @@
 <!-- TODO(lwalter) pass these in as args -->
 <xacro:include filename="$(find popcanbot_description)/urdf/popcanbot.gazebo"/>
-<!-- don't use macro names that are the same as other key names
-  like 'box', 'cylinder', etc. otherwise get Invalid parameter "size"
--->
-<xacro:macro name="block" params="name length width height mass
-    x:=0 y:=0 z:=0 r:=0.5 b:=0.5 g:=0.5">
-  <link name="${name}">
-     <visual>
-      <origin xyz="${x} ${y} ${z}" rpy="0 0 0"/>
-      <geometry>
-        <box size="${length} ${width} ${height}"/>
-      </geometry>
-      <material name="${name}_gray">
-        <color rgba="${r} ${g} ${b} 1"/>
-      </material>
-    </visual>
-    <collision>
-      <origin xyz="${x} ${y} ${z}" rpy="0 0 0"/>
-      <geometry>
-        <box size="${length} ${width} ${height}"/>
-      </geometry>
-    </collision>
-    <inertial>
-      <origin xyz="${x} ${y} ${z}" rpy="0 0 0"/>
-      <mass value="${mass}"/>
-      <inertia
-          ixx="${mass / 12.0 * (width * width + height * height)}" ixy="0.0" ixz="0.0"
-          iyy="${mass / 12.0 * (length * length + height * height)}" iyz="0.0"
-          izz="${mass / 12.0 * (length * length + width * width)}" />
-    </inertial>
-  </link>
-</xacro:macro>
-<!-- a wheel that rotates around the y axis, rolls forward toward the x axis -->
-<!--origin xyz="${length/2} ${width/2} ${height/2}" /-->
-<xacro:macro name="wheel" params="name width radius mass">
-  <link name="${name}">
-    <visual>
-      <origin xyz="0 0 0" rpy="${pi/2} 0 0" />
-      <geometry>
-        <cylinder length="${width}" radius="${radius}"/>
-      </geometry>
-      <material name="${name}_black">
-        <color rgba="0.2 0.2 0.2 1"/>
-      </material>
-    </visual>
-    <collision>
-      <origin xyz="0 0 0" rpy="${pi/2} 0 0" />
-      <geometry>
-        <cylinder length="${width}" radius="${radius}"/>
-      </geometry>
-    </collision>
-    <inertial>
-      <origin xyz="0 0 0" rpy="${pi/2} 0 0" />
-      <mass value="${mass}"/>
-      <inertia
-          ixx="${mass / 12.0 * (3 * radius * radius + width * width)}" ixy="0.0" ixz="0.0"
-          iyy="${mass / 12.0 * (3 * radius * radius + width * width)}" iyz="0.0"
-          izz="${mass / 2.0 * (radius * radius)}"/>
-    </inertial>
-  </link>
-</xacro:macro>
-<xacro:macro name="generic_wheel" params="name parent radius width
-    z:=0 y:=0 y_axis:=1 mass:=0.2 use_tran:=true">
-  <xacro:wheel name="${name}" width="${width}" radius="${radius}" mass="${mass}"/>
-  <joint name="${name}_joint" type="continuous">
-    <parent link="${parent}"/>
-    <child link="${name}"/>
-    <origin xyz="0 ${y} ${z}" rpy="0 0 0"/>
-    <axis xyz="0 ${y_axis} 0"/>
-    <limit effort="100.0" velocity="0.5"/>
-  </joint>
-  <xacro:if value="${use_tran}">
-  <transmission name="${name}_tran">
-    <type>transmission_interface/SimpleTransmission</type>
-    <joint name="${name}_joint">
-      <hardwareInterface>EffortJointInterface</hardwareInterface>
-    </joint>
-    <actuator name="${name}_motor">
-      <hardwareInterface>EffortJointInterface</hardwareInterface>
-      <mechanicalReduction>1</mechanicalReduction>
-    </actuator>
-  </transmission>
-  </xacro:if>
-  <gazebo reference="wheel_${name}">
-    <mu1>800</mu1>
-    <mu2>100</mu2>
-    <kp value="10000000.0"/>
-    <kd value="1.0"/>
-  </gazebo>
-</xacro:macro>  <!-- generic wheel -->
+<xacro:include filename="$(find popcanbot_description)/urdf/util.xacro"/>
   <link name="base_link"/>
   <xacro:block name="chassis_link" length="${car_length}"

Commit message: Added gripper control, mimic doesn't work in gazebo so have and independent controller and mimic it in software.

File: popcanbot_description/urdf/popcanbot.xacro (robot description, xacro)
@@ -120,13 +120,30 @@
     <origin xyz="0.25 0.02 -0.05" rpy="0 0 0"/>
     <axis xyz="0 0 1"/>
-    <limit effort="100.0" upper="0.4" lower="-0.1" velocity="0.5"/>
-  </joint>
-  <xacro:block name="gripper_left_tip" length="0.07"
+    <limit effort="100.0" upper="0.7" lower="-0.1" velocity="0.5"/>
+  </joint>
+  <xacro:block name="gripper_left_mid" length="0.07"
+      width="0.02" height="0.02" mass="0.05" r="0.1" b="0.1" g="0.6" x="0.03"/>
+  <joint name="gripper_left_mid_joint" type="fixed">
+    <parent link="gripper_left"/>
+    <child link="gripper_left_mid"/>
+    <origin xyz="0.05 0.0 0.0" rpy="0 0 -0.3"/>
+  </joint>
+  <xacro:block name="gripper_left_tip" length="0.05"
       width="0.02" height="0.02" mass="0.05" r="0.1" b="0.1" g="0.6" x="0.03"/>
   <joint name="gripper_left_tip_joint" type="fixed">
-    <parent link="gripper_left"/>
+    <parent link="gripper_left_mid"/>
     <child link="gripper_left_tip"/>
     <origin xyz="0.05 0.0 0.0" rpy="0 0 -0.3"/>
   </joint>
+  <transmission name="gripper_left_rotary_tran">
+    <type>transmission_interface/SimpleTransmission</type>
+    <joint name="gripper_left_joint">
+      <hardwareInterface>EffortJointInterface</hardwareInterface>
+    </joint>
+    <actuator name="gripper_left_motor">
+      <hardwareInterface>EffortJointInterface</hardwareInterface>
+      <mechanicalReduction>1</mechanicalReduction>
+    </actuator>
+  </transmission>
   <xacro:block name="gripper_right" length="0.07"
       width="0.02" height="0.02" mass="0.05" r="0.1" b="0.1" g="0.6" x="0.03"/>
@@ -137,9 +154,17 @@
     <axis xyz="0 0 1"/>
     <limit effort="100.0" upper="0.1" lower="-0.4" velocity="0.5"/>
-  </joint>
-  <xacro:block name="gripper_right_tip" length="0.07"
+    <mimic joint="gripper_left_joint" multiplier="-1.0"/>
+  </joint>
+  <xacro:block name="gripper_right_mid" length="0.07"
+      width="0.02" height="0.02" mass="0.05" r="0.1" b="0.1" g="0.6" x="0.03"/>
+  <joint name="gripper_right_mid_joint" type="fixed">
+    <parent link="gripper_right"/>
+    <child link="gripper_right_mid"/>
+    <origin xyz="0.05 0.0 0.0" rpy="0 0 0.3"/>
+  </joint>
+  <xacro:block name="gripper_right_tip" length="0.05"
       width="0.02" height="0.02" mass="0.05" r="0.1" b="0.1" g="0.6" x="0.03"/>
   <joint name="gripper_right_tip_joint" type="fixed">
-    <parent link="gripper_right"/>
+    <parent link="gripper_right_mid"/>
     <child link="gripper_right_tip"/>
     <origin xyz="0.05 0.0 0.0" rpy="0 0 0.3"/>
@@ -161,5 +186,5 @@
     <parent link="camera_mast"/>
     <child link="camera_link"/>
-    <origin xyz="0.0 0 0.0" rpy="0 0.4 0"/>
+    <origin xyz="0.0 0 0.0" rpy="0 0.6 0"/>
   </joint>
   <link name="camera_link_optical"/>
