Commit message: Added actuator for right half of gripper, shrink down coke can to a third of default size

File: popcanbot_description/urdf/popcanbot.xacro (robot description, xacro)
@@ -154,4 +154,5 @@
     <axis xyz="0 0 1"/>
     <limit effort="100.0" upper="0.1" lower="-0.4" velocity="0.5"/>
+    <!-- mimic doesn't do anything in gazebo, but should be useful in pure rviz -->
     <mimic joint="gripper_left_joint" multiplier="-1.0"/>
   </joint>
@@ -170,4 +171,14 @@
     <origin xyz="0.05 0.0 0.0" rpy="0 0 0.3"/>
   </joint>
+  <transmission name="gripper_right_rotary_tran">
+    <type>transmission_interface/SimpleTransmission</type>
+    <joint name="gripper_right_joint">
+      <hardwareInterface>EffortJointInterface</hardwareInterface>
+    </joint>
+    <actuator name="gripper_right_motor">
+      <hardwareInterface>EffortJointInterface</hardwareInterface>
+      <mechanicalReduction>1</mechanicalReduction>
+    </actuator>
+  </transmission>
   <!-- sensors -->
   <xacro:if value="${use_camera}">

Commit message: Reasonable cmd_vel to joint state + odometry tf publish, but also need to pass in proper base_radius and wheel_radius values so urdf matches.  Would like to visualize spin center and projected motion forward and back like in carbot.

File: popcanbot_description/urdf/popcanbot.xacro (robot description, xacro)
@@ -19,5 +19,5 @@
     <parent link="base_link"/>
     <child link="chassis_link"/>
-    <origin xyz="0 0 0" rpy="0 0 0"/>
+    <origin xyz="${-car_length/2 + 0.05} 0 0" rpy="0 0 0"/>
   </joint>
   <!-- every link has to have inertia in order for it to work in gazebo
@@ -31,5 +31,5 @@
     <child link="caster_block"/>
     <axis xyz="0 0 1"/>
-    <origin xyz="${-car_length/2 + 0.1} 0 ${-car_height/2}" rpy="0 0 0"/>
+    <origin xyz="${-car_length + 0.1} 0 ${-car_height/2}" rpy="0 0 0"/>
   </joint>
   <xacro:generic_wheel name="wheel_caster" parent="caster_block"
@@ -43,5 +43,5 @@
     <parent link="base_link"/>
     <child link="main_axle"/>
-    <origin xyz="${car_length/2 - 0.1} 0 ${-(car_height/2 + clearance - wheel_radius)}"
+    <origin xyz="0 0 ${-(car_height/2 + clearance - wheel_radius)}"
         rpy="0 0 0"/>
   </joint>
@@ -59,5 +59,5 @@
     <parent link="base_link"/>
     <child link="arm_vertical"/>
-    <origin xyz="0 0 ${car_height/4}" rpy="0 0 0"/>
+    <origin xyz="${-car_length/3} 0 ${car_height/4}" rpy="0 0 0"/>
     <axis xyz="0 0 1"/>
     <limit effort="100.0" upper="1.6" lower="-1.6" velocity="0.5"/>

Commit message: Have front sonar work (it detects the gripper and arm), but the cmd_vel_to_joint_state node isn't running

File: popcanbot_description/urdf/popcanbot.xacro (robot description, xacro)
@@ -210,3 +210,10 @@
   </joint>
   </xacro:if>
+  <xacro:block name="sonar_link" length="0.015"
+      width="0.05" height="0.02" mass="0.1"/>
+  <joint name="sonar_joint" type="fixed">
+    <parent link="base_link"/>
+    <child link="sonar_link"/>
+    <origin xyz="0.05 0 0.05" rpy="0 -0.1 0"/>
+  </joint>
 </robot>

Commit message: Ran into same old controller_manager inability to load robot_description outside of / https://github.com/ros-simulation/gazebo_ros_pkgs/issues/112 and http://answers.ros.org/question/198929/running-controller_manager-spawner-with-mybotrobot_description/, which is apparently fixed, but not in released packages?  Need to follow up with that.
Made the pop can bigger but now it doesn't spawn in the fridge, maybe should just make own cylinder object with a xacro and all so it can be controlled better, just make it solid red.

Was running into problems with two joint_state_publishers (though the namespace solution above would solve it, if it actually is working?), so disabled the fridge joint_state_publisher.

The friction coefficients work okay but not great, still need to drive very slowly.

File: popcanbot_description/urdf/popcanbot.xacro (robot description, xacro)
@@ -36,5 +36,7 @@
       width="${wheel_width}"
       radius="${caster_wheel_radius}" mass="0.1" use_tran="false"
-      z="${-(clearance - caster_wheel_radius)}"/>
+      x="0.02"
+      z="${-(clearance - caster_wheel_radius)}"
+      mu1="20" mu2="10"/>
   <xacro:block name="main_axle" length="${car_width/8.0}"
       width="${car_width + 0.05}" height="${car_width/8.0}" mass="0.1"
@@ -118,5 +120,5 @@
     <parent link="arm_horizontal"/>
     <child link="gripper_left"/>
-    <origin xyz="0.25 0.02 -0.05" rpy="0 0 0"/>
+    <origin xyz="0.25 0.02 -0.1" rpy="0 0 0"/>
     <axis xyz="0 0 1"/>
     <limit effort="100.0" upper="0.7" lower="-0.1" velocity="0.5"/>
@@ -151,5 +153,5 @@
     <parent link="arm_horizontal"/>
     <child link="gripper_right"/>
-    <origin xyz="0.25 -0.02 -0.05" rpy="0 0 0"/>
+    <origin xyz="0.25 -0.02 -0.1" rpy="0 0 0"/>
     <axis xyz="0 0 1"/>
     <limit effort="100.0" upper="0.1" lower="-0.4" velocity="0.5"/>

File: popcanbot_description/urdf/util.xacro (robot description, xacro)
@@ -62,10 +62,12 @@
 </xacro:macro>
 <xacro:macro name="generic_wheel" params="name parent radius width
-    z:=0 y:=0 y_axis:=1 mass:=0.2 use_tran:=true">
+    x:=0 y:=0 z:=0
+    y_axis:=1 mass:=0.2 use_tran:=true
+    mu1:=200 mu2:=100">
   <xacro:wheel name="${name}" width="${width}" radius="${radius}" mass="${mass}"/>
   <joint name="${name}_joint" type="continuous">
     <parent link="${parent}"/>
     <child link="${name}"/>
-    <origin xyz="0 ${y} ${z}" rpy="0 0 0"/>
+    <origin xyz="${x} ${y} ${z}" rpy="0 0 0"/>
     <axis xyz="0 ${y_axis} 0"/>
     <limit effort="100.0" velocity="0.5"/>
@@ -83,7 +85,7 @@
   </transmission>
   </xacro:if>
-  <gazebo reference="wheel_${name}">
-    <mu1>800</mu1>
-    <mu2>100</mu2>
+  <gazebo reference="${name}">
+    <mu1>${mu1}</mu1>
+    <mu2>${mu2}</mu2>
     <kp value="10000000.0"/>
     <kd value="1.0"/>

Commit message: #1 diff drive controller doesn't slide and go backwards like raw wheel simulation, other difference is that negative z is a left spin which has some intuitive sense but seems wrong given the standard ros robot coordinate convention- but surely move_base works with this so it must be consistent?

File: popcanbot_description/urdf/popcanbot.xacro (robot description, xacro)
@@ -5,4 +5,5 @@
 <xacro:property name="car_height" value="0.05"/>
 <xacro:property name="clearance" value="0.10"/>
+<xacro:property name="wheel_separation" value="0.56"/>
 <xacro:property name="wheel_width" value="0.025"/>
 <xacro:property name="wheel_radius" value="0.07"/>
@@ -49,10 +50,11 @@
   </joint>
   <xacro:generic_wheel name="wheel_front_left" parent="main_axle"
-      y="${car_width/2 + wheel_width/2 + 0.02}"
-      width="${wheel_width}" radius="${wheel_radius}"/>
+      y="${wheel_separation/2}"
+      width="${wheel_width}" radius="${wheel_radius}"
+      use_tran="false"/>
   <xacro:generic_wheel name="wheel_front_right" parent="main_axle"
-      y="${-1 * (car_width/2 + wheel_width/2 + 0.02)}"
+      y="${-wheel_separation/2}"
       width="${wheel_width}" radius="${wheel_radius}"
-      y_axis="1"/>
+      y_axis="1" use_tran="false"/>
   <!-- the arm -->
   <xacro:block name="arm_vertical" length="0.05"

Commit message: have static tf for map to odom (odom is provided by diff drive controller.

File: popcanbot_description/urdf/popcanbot.xacro (robot description, xacro)
@@ -85,5 +85,5 @@
     <origin xyz="0.05 0 0.25" rpy="0 0 0"/>
     <axis xyz="0 0 1"/>
-    <limit effort="20.0" velocity="0.25" lower="-0.14" upper="0.20"/>
+    <limit effort="20.0" velocity="0.25" lower="-0.14" upper="0.30"/>
   </joint>
   <transmission name="arm_vertical_rotary_tran">

Commit message: Made grippers into xacro block, though launching just the description results in TypeError: updateSliders() takes exactly 2 arguments (1 given)  unless use_joint_gui is false.

File: popcanbot_description/urdf/popcanbot.xacro (robot description, xacro)
@@ -120,80 +120,63 @@
   </transmission>
   <!-- gripper -->
-  <xacro:block name="gripper_left" length="0.07"
-      width="0.02" height="0.02" mass="0.05" r="0.1" b="0.1" g="0.6" x="0.03"
-      mu="1.0"/>
-  <joint name="gripper_left_joint" type="revolute">
-    <parent link="arm_horizontal"/>
-    <child link="gripper_left"/>
-    <origin xyz="0.25 0.02 -0.1" rpy="0 0 0"/>
-    <axis xyz="0 0 1"/>
-    <limit effort="200.0" upper="0.7" lower="-0.1" velocity="0.5"/>
-    <dynamics damping="0.1" friction="0.1"/>
-  </joint>
-  <xacro:block name="gripper_left_mid" length="0.07"
-      width="0.02" height="0.02" mass="0.05" r="0.1" b="0.1" g="0.6" x="0.03"
-      mu="1.0"/>
-  <joint name="gripper_left_mid_joint" type="fixed">
-    <parent link="gripper_left"/>
-    <child link="gripper_left_mid"/>
-    <origin xyz="0.05 0.0 0.0" rpy="0 0 -0.3"/>
-  </joint>
-  <xacro:block name="gripper_left_tip" length="0.05"
-      width="0.02" height="0.02" mass="0.05" r="0.1" b="0.1" g="0.6" x="0.03"
-      mu="1.0"/>
-  <joint name="gripper_left_tip_joint" type="fixed">
-    <parent link="gripper_left_mid"/>
-    <child link="gripper_left_tip"/>
-    <origin xyz="0.05 0.0 0.0" rpy="0 0 -0.3"/>
-  </joint>
-  <transmission name="gripper_left_rotary_tran">
-    <type>transmission_interface/SimpleTransmission</type>
-    <joint name="gripper_left_joint">
-      <hardwareInterface>EffortJointInterface</hardwareInterface>
-    </joint>
-    <actuator name="gripper_left_motor">
-      <hardwareInterface>EffortJointInterface</hardwareInterface>
-      <mechanicalReduction>1</mechanicalReduction>
-    </actuator>
-  </transmission>
-  <xacro:block name="gripper_right" length="0.07"
-      width="0.02" height="0.02" mass="0.05" r="0.1" b="0.1" g="0.6" x="0.03"
-      mu="1.0"/>
-  <joint name="gripper_right_joint" type="revolute">
-    <parent link="arm_horizontal"/>
-    <child link="gripper_right"/>
-    <origin xyz="0.25 -0.02 -0.1" rpy="0 0 0"/>
-    <axis xyz="0 0 1"/>
-    <limit effort="200.0" upper="0.1" lower="-0.5" velocity="0.5"/>
-    <dynamics damping="0.1" friction="0.1"/>
-    <!-- mimic doesn't do anything in gazebo, but should be useful in pure rviz -->
-    <!--mimic joint="gripper_left_joint" multiplier="-1.0"/-->
-  </joint>
-  <xacro:block name="gripper_right_mid" length="0.07"
-      width="0.02" height="0.02" mass="0.05" r="0.1" b="0.1" g="0.6" x="0.03"
-      mu="1.0"/>
-  <joint name="gripper_right_mid_joint" type="fixed">
-    <parent link="gripper_right"/>
-    <child link="gripper_right_mid"/>
-    <origin xyz="0.05 0.0 0.0" rpy="0 0 0.3"/>
-  </joint>
-  <xacro:block name="gripper_right_tip" length="0.05"
-      width="0.02" height="0.02" mass="0.05" r="0.1" b="0.1" g="0.6" x="0.03"
-      mu="1.0"/>
-  <joint name="gripper_right_tip_joint" type="fixed">
-    <parent link="gripper_right_mid"/>
-    <child link="gripper_right_tip"/>
-    <origin xyz="0.05 0.0 0.0" rpy="0 0 0.3"/>
-  </joint>
-  <transmission name="gripper_right_rotary_tran">
-    <type>transmission_interface/SimpleTransmission</type>
-    <joint name="gripper_right_joint">
-      <hardwareInterface>EffortJointInterface</hardwareInterface>
-    </joint>
-    <actuator name="gripper_right_motor">
-      <hardwareInterface>EffortJointInterface</hardwareInterface>
-      <mechanicalReduction>1</mechanicalReduction>
-    </actuator>
-  </transmission>
+  <xacro:macro name="gripper" params="name parent x y z roll pitch yaw ax ay az lower_lim upper_lim">
+  <xacro:block name="${name}" length="0.04"
+      width="0.02" height="0.02" mass="0.05" r="0.1" b="0.1" g="0.6" x="0.03"
+      mu="1.0"/>
+  <joint name="${name}_joint" type="revolute">
+    <parent link="${parent}"/>
+    <child link="${name}"/>
+    <origin xyz="${x} ${y} ${z}" rpy="${roll} ${pitch} ${yaw}"/>
+    <axis xyz="${ax} ${ay} ${az}"/>
+    <limit effort="200.0" upper="${upper_lim}" lower="${lower_lim}" velocity="0.5"/>
+    <dynamics damping="0.1" friction="0.1"/>
+  </joint>
+  <xacro:block name="${name}_mid1" length="0.04"
+      width="0.02" height="0.02" mass="0.05" r="0.1" b="0.1" g="0.6" x="0.03"
+      mu="1.0"/>
+  <joint name="${name}_mid1_joint" type="fixed">
+    <parent link="${name}"/>
+    <child link="${name}_mid1"/>
+    <origin xyz="0.03 0.0 0.0" rpy="0 0 -0.28"/>
+  </joint>
+  <xacro:block name="${name}_mid2" length="0.04"
+      width="0.02" height="0.02" mass="0.05" r="0.1" b="0.1" g="0.6" x="0.03"
+      mu="1.0"/>
+  <joint name="${name}_mid2_joint" type="fixed">
+    <parent link="${name}_mid1"/>
+    <child link="${name}_mid2"/>
+    <origin xyz="0.03 0.0 0.0" rpy="0 0 -0.28"/>
+  </joint>
+  <xacro:block name="${name}_tip" length="0.04"
+      width="0.02" height="0.02" mass="0.05" r="0.1" b="0.1" g="0.6" x="0.03"
+      mu="1.0"/>
+  <joint name="${name}_tip_joint" type="fixed">
+    <parent link="${name}_mid2"/>
+    <child link="${name}_tip"/>
+    <origin xyz="0.03 0.0 0.0" rpy="0 0 -0.28"/>
+  </joint>
+  <transmission name="${name}_rotary_tran">
+    <type>transmission_interface/SimpleTransmission</type>
+    <joint name="${name}_joint">
+      <hardwareInterface>EffortJointInterface</hardwareInterface>
+    </joint>
+    <actuator name="${name}_motor">
+      <hardwareInterface>EffortJointInterface</hardwareInterface>
+      <mechanicalReduction>1</mechanicalReduction>
+    </actuator>
+  </transmission>
+  </xacro:macro>
+  <xacro:gripper name="gripper_left"
+      parent="arm_horizontal"
+      x="0.25" y="0.02" z="-0.1"
+      roll="0" pitch="0" yaw="0.4"
+      ax="0" ay="0" az="-1"
+      lower_lim="-0.5" upper_lim="0.0"/>
+  <xacro:gripper name="gripper_right"
+      parent="arm_horizontal"
+      x="0.25" y="-0.02" z="-0.1"
+      roll="${pi}" pitch="0" yaw="-0.4"
+      ax="0" ay="0" az="-1"
+      lower_lim="0.0" upper_lim="5.0"/>
   <!-- sensors -->
   <xacro:if value="${use_camera}">

Commit message: Moving dr config into description so same parameters can be put into it and xacro

File: popcanbot_description/urdf/popcanbot.xacro (robot description, xacro)
@@ -10,4 +10,8 @@
 <xacro:property name="caster_wheel_radius" value="0.04"/>
 <xacro:property name="use_camera" value="true"/>
+<xacro:property name="gripper_left_lower_lim" value="-0.5"/>
+<xacro:property name="gripper_left_upper_lim" value="0.0"/>
+<xacro:property name="gripper_right_lower_lim" value="-0.5"/>
+<xacro:property name="gripper_right_upper_lim" value="0.0"/>
 <!-- TODO(lwalter) pass these in as args -->
 <xacro:include filename="$(find popcanbot_description)/urdf/popcanbot.gazebo"/>
@@ -169,14 +173,14 @@
   <xacro:gripper name="gripper_left"
       parent="arm_horizontal"
-      x="0.25" y="0.02" z="-0.1"
-      roll="0" pitch="0" yaw="0.4"
-      ax="0" ay="0" az="-1"
-      lower_lim="-0.5" upper_lim="0.0"/>
+      x="0.25" y="0.013" z="-0.1"
+      roll="0" pitch="0" yaw="0.9"
+      ax="0" ay="0" az="1"
+      lower_lim="${gripper_left_lower_lim}" upper_lim="${gripper_left_upper_lim}"/>
   <xacro:gripper name="gripper_right"
       parent="arm_horizontal"
-      x="0.25" y="-0.02" z="-0.1"
-      roll="${pi}" pitch="0" yaw="-0.4"
-      ax="0" ay="0" az="-1"
-      lower_lim="0.0" upper_lim="5.0"/>
+      x="0.25" y="-0.013" z="-0.1"
+      roll="${pi}" pitch="0" yaw="-0.9"
+      ax="0" ay="0" az="1"
+      lower_lim="${gripper_right_lower_lim}" upper_lim="${gripper_right_upper_lim}"/>
   <!-- sensors -->
   <xacro:if value="${use_camera}">
