Commit message: Have a xacro popcan spawning now, need to adjust xyz to get it into fridge.

File: popcanbot_description/urdf/popcan.xacro (robot description, xacro)
@@ -5,5 +5,5 @@
 <xacro:include filename="$(find popcanbot_description)/urdf/util.xacro"/>
   <link name="popcan_base_link"/>
-  <xacro:generic_wheel name="popcan"
+  <xacro:wheel name="popcan"
       radius="${radius}" width="${height}" mass="0.37"
       r="1.0" g="0.1" b="0.1"/>
@@ -11,5 +11,5 @@
     <parent link="popcan_base_link"/>
     <child link="popcan"/>
-    <origin xyz="0 0 0" rpy="0 ${pi/2.0} 0"/>
+    <origin xyz="0 0 0" rpy="${pi/2.0} 0 0"/>
   </joint>
 </robot>

File: popcanbot_description/urdf/util.xacro (robot description, xacro)
@@ -5,5 +5,6 @@
 -->
 <xacro:macro name="block" params="name length width height mass
-    x:=0 y:=0 z:=0 r:=0.5 b:=0.5 g:=0.5">
+    x:=0 y:=0 z:=0
+    r:=0.5 b:=0.5 g:=0.5">
   <link name="${name}">
      <visual>
@@ -34,5 +35,6 @@
 <!-- a wheel that rotates around the y axis, rolls forward toward the x axis -->
 <!--origin xyz="${length/2} ${width/2} ${height/2}" /-->
-<xacro:macro name="wheel" params="name width radius mass">
+<xacro:macro name="wheel" params="name width radius mass
+    r:=0.5 b:=0.5 g:=0.5">
   <link name="${name}">
     <visual>
@@ -42,5 +44,5 @@
       </geometry>
       <material name="${name}_black">
-        <color rgba="0.2 0.2 0.2 1"/>
+        <color rgba="${r} ${g} ${b} 1"/>
       </material>
     </visual>
@@ -60,10 +62,15 @@
     </inertial>
   </link>
+  <gazebo reference="${name}">
+    <color rgba="${r} ${g} ${b} 1.0"/>
+  </gazebo>
 </xacro:macro>
 <xacro:macro name="generic_wheel" params="name parent radius width
     x:=0 y:=0 z:=0
+    r:=0.6 g:=0.6 b:=0.6
     y_axis:=1 mass:=0.2 use_tran:=true
     mu1:=200 mu2:=100">
-  <xacro:wheel name="${name}" width="${width}" radius="${radius}" mass="${mass}"/>
+  <xacro:wheel name="${name}" width="${width}" radius="${radius}" mass="${mass}"
+      r="1.0" g="1.0" b="1.0"/>
   <joint name="${name}_joint" type="continuous">
     <parent link="${parent}"/>

Commit message: Try out a slightly conical popcan, increase friction

File: popcanbot_description/urdf/popcan.xacro (robot description, xacro)
@@ -3,14 +3,52 @@
 <xacro:property name="radius" value="0.027051"/>
 <xacro:property name="height" value="0.122682"/>
+<xacro:property name="mu" value="5.0"/>
 <xacro:include filename="$(find popcanbot_description)/urdf/util.xacro"/>
+  <!-- Make a slightly conical cylinder to increase ability to hold can -->
   <link name="popcan_base_link"/>
-  <xacro:wheel name="popcan"
-      radius="${radius}" width="${height}" mass="0.37"
+  <xacro:wheel name="popcan1"
+      radius="${radius}" width="${height/5.0}" mass="${0.37/5.0}"
       r="1.0" g="0.1" b="0.1"
-      mu="1.0"/>
-  <joint name="bottom_joint" type="fixed">
+      mu="${mu}"/>
+  <joint name="popcan_joint1" type="fixed">
     <parent link="popcan_base_link"/>
-    <child link="popcan"/>
+    <child link="popcan1"/>
     <origin xyz="0 0 0" rpy="${pi/2.0} 0 0"/>
   </joint>
+  <xacro:wheel name="popcan2"
+      radius="${radius + 0.0001}" width="${height/5.0}" mass="${0.37/5.0}"
+      r="1.0" g="0.1" b="0.1"
+      mu="${mu}"/>
+  <joint name="popcan_joint2" type="fixed">
+    <parent link="popcan1"/>
+    <child link="popcan2"/>
+    <origin xyz="0 ${height/5.0} 0" rpy="0 0 0"/>
+  </joint>
+  <xacro:wheel name="popcan3"
+      radius="${radius + 0.0002}" width="${height/5.0}" mass="${0.37/5.0}"
+      r="1.0" g="0.1" b="0.1"
+      mu="${mu}"/>
+  <joint name="popcan_joint3" type="fixed">
+    <parent link="popcan2"/>
+    <child link="popcan3"/>
+    <origin xyz="0 ${height/5.0} 0" rpy="0 0 0"/>
+  </joint>
+  <xacro:wheel name="popcan4"
+      radius="${radius + 0.0003}" width="${height/5.0}" mass="${0.37/5.0}"
+      r="1.0" g="0.1" b="0.1"
+      mu="${mu}"/>
+  <joint name="popcan_joint4" type="fixed">
+    <parent link="popcan3"/>
+    <child link="popcan4"/>
+    <origin xyz="0 ${height/5.0} 0" rpy="0 0 0"/>
+  </joint>
+  <xacro:wheel name="popcan5"
+      radius="${radius + 0.0004}" width="${height/5.0}" mass="${0.37/5.0}"
+      r="1.0" g="0.1" b="0.1"
+      mu="${mu}"/>
+  <joint name="popcan_joint5" type="fixed">
+    <parent link="popcan4"/>
+    <child link="popcan5"/>
+    <origin xyz="0 ${height/5.0} 0" rpy="0 0 0"/>
+  </joint>
 </robot>
